File: exp-1/$exp-1.sch (KiCad schematic (older format))
At the start: 87 parts, among them P1 CONN_2, P2 CONN_2, P3 CONN_2, Q1 2n5109, U1 ABA-52563, U2 AVT-50663, U3 ABA-52563, U4 AVT-50663

Commit message: Continued work on radio project thing
Parts:
- removed P1: CONN_2, symbol CONN_2
- added SL1: SDRSEL, exp-1:BSEL2, symbol SDRSEL
- added U5: ADE-1, exp-1:PL-052, symbol ADE-1
Connections:
- net GND: now also U5.1, U5.4, U5.5
- net TX_P: now also SL1.1; no longer P3.1 (P1)
- net at C10.1: now also U5.3 (RF)
- net at D2.1, L13.1: now also C31.2; no longer C31.1
- new net: P3.1 (P1), SL1.2
- new net IF: U5.2 (IF)
- new net LO: U5.6 (LO)
- new net TX_SL: C31.1, SL1.3
Other:
- moved on the sheet: C31, P3
