File: exp-1/_autosave-exp-1.kicad_pcb (KiCad board)
At the start: 4 copper layers, 50.8 x 50.8 mm, 128 parts, among them P1 CONN_8, Q1 2n5109, Q2 MMBT3904T, Q3 MMBT3904T, Q4 DMP3099L, Q5 MMBT3904T, Q6 DMP3099L, U1 ABA-52563, U2 AVT-50663, U3 ABA-52563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

Commit message: Schematic probably done. Layout still needs work
Parts:
- added P2: BNC, Connect:bnc-ci, F.Cu at (115.4, 165.2)
- added P4: BNC, exp-1:TE_BNC_VERT, F.Cu at (120.9, 122.9)
Connections:
- FILT3 pad 3: /RATT_2 -> /RATT2
Routing:
- net /RATT_2: track 53.6 -> 45.6 mm
- net /RATT2: track 0.00 -> 7.98 mm
